File: schematic_seperate_gnd.brd (EAGLE design)
At the start: 83.5 x 80 mm, 48 parts, among them U1 FT232RL-BASICSSOP

Commit message: inital routing complete
Parts:
- moved VIN 1.42 mm to (1.91, 78.1)
- moved RESET 1.27 mm to (4.45, 5.08)
- moved SWIN 1.27 mm to (4.45, 20.3)
Connections:
- new net AGND: ADC.4, C4.2, C5.2, C8.2, C9.2, D2.K, DAC.3, R10.P$1, R8.P$1, U1.25, VIN.2, VTEST.2
- net GND: no longer ADC.4, C4.2, C5.2, C8.2, C9.2, D2.K, DAC.3, R10.P$1, R8.P$1, U1.25, VIN.2, VTEST.2
Routing:
- net GND: track 105.2 -> 29.5 mm, vias 3 -> 0
- net AGND: track 0.00 -> 57.7 mm, vias 0 -> 2
- net VCC: track 24.0 -> 13.2 mm, vias 1 -> 0
- net N$11: track 14.2 -> 15.9 mm
- net ~RST: track 68.4 -> 69.6 mm
- net MSP_SWIN: track 44.7 -> 45.8 mm
- removed copper zone on layer 16, net GND
- removed copper zone on layer 1, net VCC
