File: schematic_seperate_gnd.sch (EAGLE design)
At the start: 48 parts, among them U1 FT232RL-BASICSSOP

Commit message: inital routing complete
Connections:
- new net AGND: ADC.GND, C4.2, C5.2, C8.2, C9.2, D2.C, DAC.GND, R10.1, R8.1, U1.AGND, VIN.2, VTEST.2
- net GND: no longer ADC.GND, C4.2, C5.2, C8.2, C9.2, D2.C, DAC.GND, R10.1, R8.1, U1.AGND, VIN.2, VTEST.2
